File: _autosave-NuisanceEngine.kicad_pcb (KiCad board)
At the start: 2 copper layers, 58 x 53 mm, 59 parts, among them J1 CV, J2 Headphones, J3 Power, Q1 2N3904, Q2 2N3904, Q3 TIP31A, Q4 TIP32A, SW1 SW_SPDT, SW2 SW_SPDT, U1 LM324

Commit message: gonna rearrange shit to allow for clean transistor placement
Parts:
- moved Q3 12.1 mm to (69.0, 50.0), turned to 270 degrees
- moved Q4 10.9 mm to (74.0, 55.0), turned to 90 degrees
Routing:
- net Net-(R2-Pad1): track 7.35 -> 0.00 mm
- net VDD: track 61.7 -> 57.2 mm
Changed lines of the file:
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@@
     (thickness 1.6)
     (drawings 53)
-    (tracks 336)
+    (tracks 328)
     (zones 0)
     (modules 59)
@@
     (35 F.Paste user hide)
     (36 B.SilkS user)
-    (37 F.SilkS user hide)
+    (37 F.SilkS user)
     (38 B.Mask user)
-    (39 F.Mask user hide)
+    (39 F.Mask user)
     (40 Dwgs.User user)
     (41 Cmts.User user)
@@
   )
   (setup
-    (last_trace_width 0.25)
+    (last_trace_width 1)
     (user_trace_width 0.5)
     (user_trace_width 1)
@@
   )
   (module Package_TO_SOT_THT:TO-220-3_Vertical (layer B.Cu)
-    (at 63.5 52 180)
+    (at 74 55 90)
     (descr "TO-220-3, Vertical, RM 2.54mm, see https://www.vishay.com/docs/66542/to-220-1.pdf")
     (tags "TO-220-3 Vertical RM 2.54mm")
-    (fp_text reference Q4 (at 8.5 0 90) (layer B.SilkS)
+    (fp_text reference Q4 (at 8.5 0) (layer B.SilkS)
       (effects (font (size 1 1) (thickness 0.15)) (justify mirror))
     )
-    (fp_text value TIP32A (at 2.54 -2.5 180) (layer B.Fab)
+    (fp_text value TIP32A (at 2.54 -2.5 270) (layer B.Fab)
       (effects (font (size 1 1) (thickness 0.15)) (justify mirror))
     )
-    (fp_text user %R (at 2.54 4.27 180) (layer B.Fab)
+    (fp_text user %R (at 2.54 4.27 270) (layer B.Fab)
       (effects (font (size 1 1) (thickness 0.15)) (justify mirror))
     )
@@
     (fp_line (start -2.46 -1.25) (end 7.54 -1.25) (layer B.Fab) (width 0.1))
     (fp_line (start -2.46 3.15) (end -2.46 -1.25) (layer B.Fab) (width 0.1))
-    (pad 3 thru_hole oval (at 5.08 0 180) (size 1.905 2) (drill 1.1) (layers *.Cu *.Mask)
+    (pad 3 thru_hole oval (at 5.08 0 90) (size 1.905 2) (drill 1.1) (layers *.Cu *.Mask)
       (net 14 "Net-(C8-Pad1)"))
-    (pad 2 thru_hole oval (at 2.54 0 180) (size 1.905 2) (drill 1.1) (layers *.Cu *.Mask)
+    (pad 2 thru_hole oval (at 2.54 0 90) (size 1.905 2) (drill 1.1) (layers *.Cu *.Mask)
       (net 1 GND))
-    (pad 1 thru_hole rect (at 0 0 180) (size 1.905 2) (drill 1.1) (layers *.Cu *.Mask)
+    (pad 1 thru_hole rect (at 0 0 90) (size 1.905 2) (drill 1.1) (layers *.Cu *.Mask)
       (net 12 "Net-(C7-Pad1)"))
     (model ${KISYS3DMOD}/Package_TO_SOT_THT.3dshapes/TO-220-3_Vertical.wrl
@@
   )
   (module Package_TO_SOT_THT:TO-220-3_Vertical (layer B.Cu)
-    (at 61.5 59.5 180)
+    (at 69 50 270)
     (descr "TO-220-3, Vertical, RM 2.54mm, see https://www.vishay.com/docs/66542/to-220-1.pdf")
     (tags "TO-220-3 Vertical RM 2.54mm")
-    (fp_text reference Q3 (at -3.5 1 90) (layer B.SilkS)
+    (fp_text reference Q3 (at -3.5 1) (layer B.SilkS)
       (effects (font (size 1 1) (thickness 0.15)) (justify mirror))
     )
-    (fp_text value TIP31A (at 2.54 -2.5 180) (layer B.Fab)
+    (fp_text value TIP31A (at 2.54 -2.5 270) (layer B.Fab)
       (effects (font (size 1 1) (thickness 0.15)) (justify mirror))
     )
-    (fp_text user %R (at 2.54 4.27 180) (layer B.Fab)
+    (fp_text user %R (at 2.54 4.27 270) (layer B.Fab)
       (effects (font (size 1 1) (thickness 0.15)) (justify mirror))
     )
@@
     (fp_line (start -2.46 -1.25) (end 7.54 -1.25) (layer B.Fab) (width 0.1))
     (fp_line (start -2.46 3.15) (end -2.46 -1.25) (layer B.Fab) (width 0.1))
-    (pad 3 thru_hole oval (at 5.08 0 180) (size 1.905 2) (drill 1.1) (layers *.Cu *.Mask)
+    (pad 3 thru_hole oval (at 5.08 0 270) (size 1.905 2) (drill 1.1) (layers *.Cu *.Mask)
       (net 14 "Net-(C8-Pad1)"))
-    (pad 2 thru_hole oval (at 2.54 0 180) (size 1.905 2) (drill 1.1) (layers *.Cu *.Mask)
+    (pad 2 thru_hole oval (at 2.54 0 270) (size 1.905 2) (drill 1.1) (layers *.Cu *.Mask)
       (net 16 VDD))
-    (pad 1 thru_hole rect (at 0 0 180) (size 1.905 2) (drill 1.1) (layers *.Cu *.Mask)
+    (pad 1 thru_hole rect (at 0 0 270) (size 1.905 2) (drill 1.1) (layers *.Cu *.Mask)
       (net 12 "Net-(C7-Pad1)"))
     (model ${KISYS3DMOD}/Package_TO_SOT_THT.3dshapes/TO-220-3_Vertical.wrl
@@
   (segment (start 61.5 68.5) (end 66.75 73.75) (width 0.5) (layer F.Cu) (net 16))
   (segment (start 61.5 62.5) (end 61.5 68.5) (width 0.5) (layer F.Cu) (net 16))
-  (segment (start 59.987499 57.799999) (end 58.96 58.827498) (width 1) (layer F.Cu) (net 16))
-  (segment (start 64.356003 57.799999) (end 59.987499 57.799999) (width 1) (layer F.Cu) (net 16))
-  (segment (start 65.600001 56.556001) (end 64.356003 57.799999) (width 1) (layer F.Cu) (net 16))
-  (segment (start 65.600001 56.039997) (end 65.600001 56.556001) (width 1) (layer F.Cu) (net 16))
-  (segment (start 58.96 58.827498) (end 58.96 59.5) (width 1) (layer F.Cu) (net 16))
-  (segment (start 66.139999 55.499999) (end 65.600001 56.039997) (width 1) (layer F.Cu) (net 16))
-  (segment (start 67.875001 55.499999) (end 66.139999 55.499999) (width 1) (layer F.Cu) (net 16))
-  (segment (start 69 54.375) (end 67.875001 55.499999) (width 1) (layer F.Cu) (net 16))
-  (segment (start 58.96 59.96) (end 61.5 62.5) (width 0.5) (layer B.Cu) (net 16))
   (segment (start 58.96 59.5) (end 58.96 59.96) (width 0.5) (layer B.Cu) (net 16))
+  (segment (start 66.639999 55.499999) (end 67.875001 55.499999) (width 1) (layer F.Cu) (net 16))
+  (segment (start 69 54.375) (end 67.875001 55.499999) (width 1) (layer F.Cu) (net 16))
+  (segment (start 66.639999 55.499999) (end 66.249999 55.889999) (width 1) (layer F.Cu) (net 16))
+  (segment (start 66.249999 55.889999) (end 66.249999 57.750001) (width 1) (layer F.Cu) (net 16))
+  (segment (start 66.249999 57.750001) (end 61.5 62.5) (width 1) (layer F.Cu) (net 16))
   (segment (start 68 98) (end 68 96.9) (width 0.25) (layer F.Cu) (net 17))
   (segment (start 75.475 95) (end 76.475 94) (width 0.25) (layer F.Cu) (net 17))
@@
   (segment (start 81.925001 81.075999) (end 81.925001 87.824999) (width 0.25) (layer B.Cu) (net 27))
   (segment (start 79.600998 79.75) (end 80.599002 79.75) (width 0.25) (layer B.Cu) (net 27))
-  (segment (start 64.625928 62.500928) (end 65.125 63) (width 0.25) (layer F.Cu) (net 28))
-  (segment (start 63.399999 61.274999) (end 64.625928 62.500928) (width 0.25) (layer F.Cu) (net 28))
-  (segment (start 60.225001 61.274999) (end 63.399999 61.274999) (width 0.25) (layer F.Cu) (net 28))
-  (segment (start 59 62.5) (end 60.225001 61.274999) (width 0.25) (layer F.Cu) (net 28))
   (segment (start 72.27 76.15) (end 72.27 75.7) (width 0.25) (layer F.Cu) (net 29))
   (segment (start 74.225001 80.710001) (end 74.225001 78.105001) (width 0.25) (layer F.Cu) (net 29))
